File: hardware/power.kicad_sch (KiCad schematic)
At the start: 0 parts

Commit message: Drew most of DC DC converters
Parts:
- added C56, C60, C61, C65, C68, C70, C73, C75, C78, C81, C84, C86: 100nF, Capacitor_SMD:C_0402_1005Metric, symbol Device:C
- added C57, C59, C66, C71, C72, C76, C77, C80, C85: 10uF, Capacitor_SMD:C_0603_1608Metric, symbol Device:C
- added C58, C63, C69, C74, C82: 22pF, Capacitor_SMD:C_0402_1005Metric, symbol Device:C
- added C62, C64, C67, C79, C83: 22uF, Capacitor_SMD:C_0603_1608Metric, symbol Device:C
- added L2, L4: 4.7uH, symbol Device:L
- added L3, L5, L6, L7: 2.2uH, symbol Device:L
- added Q3: AO3415A, Package_TO_SOT_SMD:SOT-23, symbol Transistor_FET:AO3401A
- added R38, R39, R41, R44, R46, R48: 10k, Resistor_SMD:R_0402_1005Metric, symbol Device:R
- added R40: 15k, Resistor_SMD:R_0402_1005Metric, symbol Device:R
- added R42, R43, R50: 100k, Resistor_SMD:R_0402_1005Metric, symbol Device:R
- added R45, R47, R51: 2.21k, Resistor_SMD:R_0402_1005Metric, symbol Device:R
- added R49: 33k, Resistor_SMD:R_0402_1005Metric, symbol Device:R
- added U17, U18: SY8088, Package_TO_SOT_SMD:SOT-23-5, symbol cm0:SY8088
- added U19, U20, U22: SY8089A, Package_TO_SOT_SMD:SOT-23-5, symbol cm0:SY8089A
- added U21: SY8113, Package_TO_SOT_SMD:TSOT-23-6, symbol cm0:SY8113
Connections:
- new net: C82.2, R48.1, R51.2, U22.5 (FB)
- new net: L3.1, U19.3 (LX)
- new net: C63.2, R42.1, R43.2, U19.5 (FB)
- new net: L6.1, U22.3 (LX)
- new net: L5.1, U20.3 (LX)
- new net: C74.2, R46.1, R47.2, U20.5 (FB)
- new net: L2.1, U17.3 (LX)
- new net: C58.2, R40.1, R41.2, U17.5 (FB)
- new net: C75.1, C76.2, C77.2
- new net: C69.2, R44.1, R45.2, U18.5 (FB)
- new net: L4.1, U18.3 (LX)
- new net: Q3.3 (D), R49.1, U22.1 (EN)
- new net: C78.1, L7.1, U21.6 (LX)
- new net: C78.2, U21.1 (BS)
- new net +1V2: C63.1, C64.1, C65.2, C66.1, L3.2, R42.2
- new net +1V5: C58.1, C59.1, C60.2, L2.2, R40.2
- new net +3V3_AVCC: C74.1, C75.2, C76.1, C77.1, L5.2, Q3.2 (S), R38.1, R39.1, R46.2
- new net +3V3_IO: C82.1, C83.1, C84.2, L6.2, R48.2
- new net +3V3_WIFI: C69.1, C70.2, C71.1, L4.2, R44.2
- new net +5V: C56.2, C57.1, C61.2, C62.1, C67.1, C68.2, C72.1, C73.2, C79.1, C80.1, C81.2, C85.1, C86.2, U17.4 (IN), U18.1 (EN), U18.4 (IN), U19.4 (IN), U20.1 (EN), U20.4 (IN), U21.5 (IN), U22.4 (IN)
- new net GND: C56.1, C57.2, C59.2, C60.1, C61.1, C62.2, C64.2, C65.1, C66.2, C67.2, C68.1, C70.1, C71.2, C72.2, C73.1, C79.2, C80.2, C81.1, C83.2, C84.1, C85.2, C86.1, R41.1, R43.1, R45.1, R47.1, R49.2, R50.1, R51.1, U17.2 (GND), U18.2 (GND), U19.2 (GND), U20.2 (GND), U21.2 (GND), U22.2 (GND)
- new net PWR_DRAM: R38.2, U17.1 (EN)
- new net PWR_IO: Q3.1 (G), R50.2
- new net PWR_SYSTEM: R39.2, U19.1 (EN), U21.4 (EN)
Other:
- added sheet Power Tree (power_tree.kicad_sch)
- note added: "0.6*(30/6.8+1)=3.3? 0.6*(150/33+1)=3.3?"
- note added: "Bigger unique L?"
- note added: "DRAM 1.5V/1A Vout=0.6*(1+R1/R2) Vout=0.6*(1+15/10)=1.5V"
- note added: "IO 3.3V/2A Vout=0.6*(1+R1/R2) Vout=0.6*(1+10/2.21)=3.3V"
- note added: "RTC 3.3V/2A Vout=0.6*(1+R1/R2) Vout=0.6*(1+10/2.21)=3.3V"
- note added: "SYSTEM 1.2V/2A Vout=0.6*(1+R1/R2) Vout=0.6*(1+100/100)=1.2V"
- note added: "WIFI 3.3V/1A Vout=0.6*(1+R1/R2) Vout=0.6*(1+10/2.21)=3.3V"
