File: hardware/ddr3.kicad_sch (KiCad schematic)
At the start: 22 parts, among them U2 H5TQ4G63EFR

Commit message: Improve routing and add test pads
Parts:
- U2: LCSC Part # C2803248 -> C2803259
Changed lines of the file:
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@@
 			)
 		)
-		(property "LCSC Part #" "C2803248"
+		(property "LCSC Part #" "C2803259"
 			(at 95.25 109.22 0)
 			(effects

Commit message: Production ready
Parts:
- R7, R8: value 2k -> 2.2k; LCSC Part # C4109 -> C25879
Changed lines of the file:
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@@
 			)
 		)
-		(property "Value" "2k"
+		(property "Value" "2.2k"
 			(at 152.4 67.3099 0)
 			(effects
@@
 			)
 		)
-		(property "LCSC Part #" "C4109"
+		(property "LCSC Part #" "C25879"
 			(at 154.94 66.04 0)
 			(effects
@@
 			)
 		)
-		(property "Value" "2k"
+		(property "Value" "2.2k"
 			(at 152.4 77.4699 0)
 			(effects
@@
 			)
 		)
-		(property "LCSC Part #" "C4109"
+		(property "LCSC Part #" "C25879"
 			(at 154.94 76.2 0)
 			(effects
