File: hardware/gpdi.kicad_sch (KiCad schematic)
At the start: 12 parts, among them J5 GPDI_A, Q3 BSN20, U19 UCL0524P, U20 UCL0524P, U23 UCL0524P

Commit message: Even more routing
Connections:
- net +3V3 renamed +3V3_IO
