File: hardware/gpdi.kicad_sch (KiCad schematic)
At the start: 12 parts, among them J5 GPDI_A, Q3 BSN20, U19 UCL0524P, U20 UCL0524P, U23 UCL0524P

Commit message: Production ready
Parts:
- R37, R38: value 33k -> 30k; LCSC Part # C25779 -> C25553
- R39, R40: value 2k -> 2.2k; LCSC Part # C4109 -> C25879
Changed lines of the file:
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@@
 			)
 		)
-		(property "Value" "2k"
+		(property "Value" "2.2k"
 			(at 129.286 77.47 90)
 			(effects
@@
 			)
 		)
-		(property "LCSC Part #" "C4109"
+		(property "LCSC Part #" "C25879"
 			(at 127 77.47 0)
 			(effects
@@
 			)
 		)
-		(property "Value" "33k"
+		(property "Value" "30k"
 			(at 153.416 46.99 90)
 			(effects
@@
 			)
 		)
-		(property "LCSC Part #" "C25779"
+		(property "LCSC Part #" "C25553"
 			(at 151.13 46.99 90)
 			(effects
@@
 			)
 		)
-		(property "Value" "2k"
+		(property "Value" "2.2k"
 			(at 134.366 77.47 90)
 			(effects
@@
 			)
 		)
-		(property "LCSC Part #" "C4109"
+		(property "LCSC Part #" "C25879"
 			(at 132.08 77.47 0)
 			(effects
@@
 			)
 		)
-		(property "Value" "33k"
+		(property "Value" "30k"
 			(at 139.446 46.99 90)
 			(effects
@@
 			)
 		)
-		(property "LCSC Part #" "C25779"
+		(property "LCSC Part #" "C25553"
 			(at 137.16 46.99 90)
 			(effects
