File: hardware/audio.kicad_sch (KiCad schematic)
At the start: 5 parts, among them J10 AudioJack_PJ-342

Commit message: Improve routing and add test pads
Parts:
- J10: FT Position Offset -0.3175,0.4445 -> -2.57175,-0.03175
Changed lines of the file:
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@@
 			)
 		)
-		(property "FT Position Offset" "-0.3175,0.4445"
+		(property "FT Position Offset" "-2.57175,-0.03175"
 			(at 125.73 93.98 0)
 			(effects
