File: hardware/gpio.kicad_sch (KiCad schematic)
At the start: 10 parts, among them J8 UART, J9 GPIO, Q4 BSN20

Commit message: Improve routing and add test pads
Parts:
- D3, D4: LCSC Part # C965804 -> C2290
Changed lines of the file:
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@@
 			)
 		)
-		(property "LCSC Part #" "C965804"
+		(property "LCSC Part #" "C2290"
 			(at 189.23 88.9 0)
 			(effects
@@
 			)
 		)
-		(property "LCSC Part #" "C965804"
+		(property "LCSC Part #" "C2290"
 			(at 189.23 77.47 0)
 			(effects

Commit message: Production ready
Parts:
- R71, R72: value 2k -> 2.2k; LCSC Part # C4109 -> C25879
Changed lines of the file:
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@@
 			)
 		)
-		(property "Value" "2k"
+		(property "Value" "2.2k"
 			(at 176.53 81.28 90)
 			(effects
@@
 			)
 		)
-		(property "LCSC Part #" "C4109"
+		(property "LCSC Part #" "C25879"
 			(at 177.8 88.9 0)
 			(effects
@@
 			)
 		)
-		(property "Value" "2k"
+		(property "Value" "2.2k"
 			(at 176.53 69.85 90)
 			(effects
@@
 			)
 		)
-		(property "LCSC Part #" "C4109"
+		(property "LCSC Part #" "C25879"
 			(at 177.8 77.47 0)
 			(effects
