File: hardware/wifi.kicad_sch (KiCad schematic)
At the start: 33 parts, among them J11 ANT, J7 RJ45_Hanrun_HR913550A_Horizon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, U22 AP6212, U24 AW13412HDNR, Y2 26MHz

Commit message: Improve routing and add test pads
Parts:
- J11: FT Rotation Offset (none) -> 180
- L7: LCSC Part # C19734 -> C43389
Changed lines of the file:
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@@
+			)
+		)
+		(property "FT Rotation Offset" "180"
+			(at 251.46 57.15 0)
+			(effects
+				(font
+					(size 1.27 1.27)
+				)
+				(hide yes)
 			)
 		)
@@
 			)
 		)
-		(property "LCSC Part #" "C19734"
+		(property "LCSC Part #" "C43389"
 			(at 175.26 62.23 90)
 			(effects

Commit message: Production ready
Parts:
- C115, C119, C120: value 10pF -> 15pF; LCSC Part # C32949 -> C1548
- C9: value 100pF -> 1nF; LCSC Part # C1546 -> C1523
- R46, R47, R48, R49, R50: value 33k -> 30k; LCSC Part # C25779 -> C25553
- Y2: LCSC Part # C7294683 -> C7301948
Changed lines of the file:
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@@
 			)
 		)
-		(property "Value" "10pF"
+		(property "Value" "15pF"
 			(at 186.944 73.406 90)
 			(effects
@@
 			)
 		)
-		(property "LCSC Part #" "C32949"
+		(property "LCSC Part #" "C1548"
 			(at 185.42 74.93 90)
 			(effects
@@
 			)
 		)
-		(property "Value" "33k"
+		(property "Value" "30k"
 			(at 89.916 35.56 90)
 			(effects
@@
 			)
 		)
-		(property "LCSC Part #" "C25779"
+		(property "LCSC Part #" "C25553"
 			(at 87.63 35.56 90)
 			(effects
@@
 			)
 		)
-		(property "Value" "33k"
+		(property "Value" "30k"
 			(at 105.156 35.56 90)
 			(effects
@@
 			)
 		)
-		(property "LCSC Part #" "C25779"
+		(property "LCSC Part #" "C25553"
 			(at 102.87 35.56 90)
 			(effects
@@
 			)
 		)
-		(property "Value" "33k"
+		(property "Value" "30k"
 			(at 110.236 35.56 90)
 			(effects
@@
 			)
 		)
-		(property "LCSC Part #" "C25779"
+		(property "LCSC Part #" "C25553"
 			(at 107.95 35.56 90)
 			(effects
@@
 			)
 		)
-		(property "Value" "10pF"
+		(property "Value" "15pF"
 			(at 186.944 86.614 90)
 			(effects
@@
 			)
 		)
-		(property "LCSC Part #" "C32949"
+		(property "LCSC Part #" "C1548"
 			(at 185.42 85.09 90)
 			(effects
@@
 			)
 		)
-		(property "LCSC Part #" "C7294683"
+		(property "LCSC Part #" "C7301948"
 			(at 175.26 80.01 90)
 			(effects
@@
 			)
 		)
-		(property "Value" "100pF"
+		(property "Value" "1nF"
 			(at 218.44 63.4999 0)
 			(effects
@@
 			)
 		)
-		(property "LCSC Part #" "C1546"
+		(property "LCSC Part #" "C1523"
 			(at 222.25 62.23 0)
 			(effects
@@
 			)
 		)
-		(property "Value" "33k"
+		(property "Value" "30k"
 			(at 94.996 35.56 90)
 			(effects
@@
 			)
 		)
-		(property "LCSC Part #" "C25779"
+		(property "LCSC Part #" "C25553"
 			(at 92.71 35.56 90)
 			(effects
@@
 			)
 		)
-		(property "Value" "10pF"
+		(property "Value" "15pF"
 			(at 176.53 46.99 90)
 			(effects
@@
 			)
 		)
-		(property "LCSC Part #" "C32949"
+		(property "LCSC Part #" "C1548"
 			(at 176.53 52.07 90)
 			(effects
@@
 			)
 		)
-		(property "Value" "33k"
+		(property "Value" "30k"
 			(at 100.076 35.56 90)
 			(effects
@@
 			)
 		)
-		(property "LCSC Part #" "C25779"
+		(property "LCSC Part #" "C25553"
 			(at 97.79 35.56 90)
 			(effects
